Commit message: touch up urdf naming

File: greenseeker_description/urdf/greenseeker.urdf.xacro (robot description, xacro)
@@ -38,5 +38,5 @@
         </joint>
 		<!-- sensor frame -->
-        <link name="${sensor_frame}_laser">
+        <link name="${sensor_frame}">
             <visual>
                 <origin xyz="0 0 0" rpy="0 0 0" />
@@ -49,5 +49,5 @@
         <joint name="${sensor_frame}_${name}_joint" type="fixed">
             <parent link="${name}"/>
-            <child link="${sensor_frame}_laser"/>
+            <child link="${sensor_frame}"/>
             <origin xyz="${sensor_frame_dx} ${sensor_frame_dy} ${sensor_frame_dz}" rpy="${M_PI} 0 ${M_PI/2}" />
         </joint>
